Commit message: commit at noon

File: dyros_tocabi/dyros_tocabi_parkour.urdf (robot description, URDF)
Before this commit: robot dyros_tocabi_description, 36 links, 35 joints
Links:
- link Head_Link: geometry collision box size=0.16 0.12 0.172; visual mesh filename=meshes/head.STL scale=0.001 0.001 0.001
Joints:
- joint Head_Joint: origin xyz=0.0 0.0 0.0275 rpy=0 0 0 -> xyz=0 0 0.0275 rpy=0 0 0
- joint Neck_Joint: origin xyz=-0.036 0.0 0.3795 rpy=0 0 0 -> xyz=-0.036 0 0.3795 rpy=0 0 0

Commit message: 250321_PDtune Sim setup Remove constraints Terrain setup finished TODO: wandb logging and tuning

File: dyros_tocabi/dyros_tocabi_parkour.urdf (robot description, URDF)
Before this commit: robot dyros_tocabi_description, 36 links, 35 joints
Links:
- link Pelvis_Link: geometry collision box size=0.141 0.305 0.05; collision cylinder length=0.044 radius=0.045
